File: Macropad5x5.kicad_sch (KiCad schematic)
At the start: 100 parts, among them M1 MountingHole, M2 MountingHole, M3 MountingHole, M4 MountingHole, M5 MountingHole, M6 MountingHole, M7 MountingHole, SW1 SW_Push, SW2 SW_Push, U1 PicoW, U4 SN74LV1T125DBV

Commit message: Updated 3d models.
Parts:
- MX1, MX11, MX12, MX13, MX14, MX16, MX17, MX18, MX19, MX2, MX21, MX22, MX23, MX24, MX3, MX4, MX6, MX7, MX8, MX9: footprint PCM_marbastlib-mx:SW_MX_HS_CPG151101S11_1u -> Macropad:SW_Cherry_MX_PCB_1.00u
- MX10, MX15, MX20, MX25: footprint PCM_marbastlib-mx:SW_MX_HS_CPG151101S11_1.25u -> Macropad:SW_Cherry_MX_PCB_1.25u
- MX5: footprint Rotary_Encoder:RotaryEncoder_Alps_EC11E-Switch_Vertical_H20mm -> Macropad:RotaryEncoder_Alps_EC11E-Switch_Vertical_H20mm
Changed lines of the file:
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@@
 			)
 		)
-		(property "Footprint" "PCM_marbastlib-mx:SW_MX_HS_CPG151101S11_1.25u"
+		(property "Footprint" "Macropad:SW_Cherry_MX_PCB_1.25u"
 			(at 114.3 86.36 0)
 			(effects
@@
 			)
 		)
-		(property "Footprint" "PCM_marbastlib-mx:SW_MX_HS_CPG151101S11_1u"
+		(property "Footprint" "Macropad:SW_Cherry_MX_PCB_1.00u"
 			(at 34.29 21.59 0)
 			(effects
@@
 			)
 		)
-		(property "Footprint" "PCM_marbastlib-mx:SW_MX_HS_CPG151101S11_1u"
+		(property "Footprint" "Macropad:SW_Cherry_MX_PCB_1.00u"
 			(at 34.29 86.36 0)
 			(effects
@@
 			)
 		)
-		(property "Footprint" "PCM_marbastlib-mx:SW_MX_HS_CPG151101S11_1u"
+		(property "Footprint" "Macropad:SW_Cherry_MX_PCB_1.00u"
 			(at 73.66 107.95 0)
 			(effects
@@
 			)
 		)
-		(property "Footprint" "PCM_marbastlib-mx:SW_MX_HS_CPG151101S11_1u"
+		(property "Footprint" "Macropad:SW_Cherry_MX_PCB_1.00u"
 			(at 73.66 21.59 0)
 			(effects
@@
 			)
 		)
-		(property "Footprint" "PCM_marbastlib-mx:SW_MX_HS_CPG151101S11_1u"
+		(property "Footprint" "Macropad:SW_Cherry_MX_PCB_1.00u"
 			(at 34.29 107.95 0)
 			(effects
@@
 			)
 		)
-		(property "Footprint" "PCM_marbastlib-mx:SW_MX_HS_CPG151101S11_1u"
+		(property "Footprint" "Macropad:SW_Cherry_MX_PCB_1.00u"
 			(at 73.66 86.36 0)
 			(effects
@@
 			)
 		)
-		(property "Footprint" "PCM_marbastlib-mx:SW_MX_HS_CPG151101S11_1u"
+		(property "Footprint" "Macropad:SW_Cherry_MX_PCB_1.00u"
 			(at 93.98 64.77 0)
 			(effects
@@
 			)
 		)
-		(property "Footprint" "Rotary_Encoder:RotaryEncoder_Alps_EC11E-Switch_Vertical_H20mm"
+		(property "Footprint" "Macropad:RotaryEncoder_Alps_EC11E-Switch_Vertical_H20mm"
 			(at 149.86 180.594 0)
 			(effects
@@
 			)
 		)
-		(property "Footprint" "PCM_marbastlib-mx:SW_MX_HS_CPG151101S11_1u"
+		(property "Footprint" "Macropad:SW_Cherry_MX_PCB_1.00u"
 			(at 34.29 64.77 0)
 			(effects
@@
 			)
 		)
-		(property "Footprint" "PCM_marbastlib-mx:SW_MX_HS_CPG151101S11_1u"
+		(property "Footprint" "Macropad:SW_Cherry_MX_PCB_1.00u"
 			(at 93.98 107.95 0)
 			(effects
@@
 			)
 		)
-		(property "Footprint" "PCM_marbastlib-mx:SW_MX_HS_CPG151101S11_1u"
+		(property "Footprint" "Macropad:SW_Cherry_MX_PCB_1.00u"
 			(at 53.34 107.95 0)
 			(effects
@@
 			)
 		)
-		(property "Footprint" "PCM_marbastlib-mx:SW_MX_HS_CPG151101S11_1u"
+		(property "Footprint" "Macropad:SW_Cherry_MX_PCB_1.00u"
 			(at 53.34 21.59 0)
 			(effects
@@
 			)
 		)
-		(property "Footprint" "PCM_marbastlib-mx:SW_MX_HS_CPG151101S11_1u"
+		(property "Footprint" "Macropad:SW_Cherry_MX_PCB_1.00u"
 			(at 93.98 21.59 0)
 			(effects
@@
 			)
 		)
-		(property "Footprint" "PCM_marbastlib-mx:SW_MX_HS_CPG151101S11_1u"
+		(property "Footprint" "Macropad:SW_Cherry_MX_PCB_1.00u"
 			(at 53.34 86.36 0)
 			(effects
@@
 			)
 		)
-		(property "Footprint" "PCM_marbastlib-mx:SW_MX_HS_CPG151101S11_1u"
+		(property "Footprint" "Macropad:SW_Cherry_MX_PCB_1.00u"
 			(at 93.98 43.18 0)
 			(effects
@@
 			)
 		)
-		(property "Footprint" "PCM_marbastlib-mx:SW_MX_HS_CPG151101S11_1u"
+		(property "Footprint" "Macropad:SW_Cherry_MX_PCB_1.00u"
 			(at 53.34 64.77 0)
 			(effects
@@
 			)
 		)
-		(property "Footprint" "PCM_marbastlib-mx:SW_MX_HS_CPG151101S11_1u"
+		(property "Footprint" "Macropad:SW_Cherry_MX_PCB_1.00u"
 			(at 73.66 64.77 0)
 			(effects
@@
 			)
 		)
-		(property "Footprint" "PCM_marbastlib-mx:SW_MX_HS_CPG151101S11_1u"
+		(property "Footprint" "Macropad:SW_Cherry_MX_PCB_1.00u"
 			(at 53.34 43.18 0)
 			(effects
@@
 			)
 		)
-		(property "Footprint" "PCM_marbastlib-mx:SW_MX_HS_CPG151101S11_1.25u"
+		(property "Footprint" "Macropad:SW_Cherry_MX_PCB_1.25u"
 			(at 114.3 107.95 0)
 			(effects
@@
 			)
 		)
-		(property "Footprint" "PCM_marbastlib-mx:SW_MX_HS_CPG151101S11_1u"
+		(property "Footprint" "Macropad:SW_Cherry_MX_PCB_1.00u"
 			(at 34.29 43.18 0)
 			(effects
@@
 			)
 		)
-		(property "Footprint" "PCM_marbastlib-mx:SW_MX_HS_CPG151101S11_1.25u"
+		(property "Footprint" "Macropad:SW_Cherry_MX_PCB_1.25u"
 			(at 114.3 64.77 0)
 			(effects
@@
 			)
 		)
-		(property "Footprint" "PCM_marbastlib-mx:SW_MX_HS_CPG151101S11_1u"
+		(property "Footprint" "Macropad:SW_Cherry_MX_PCB_1.00u"
 			(at 93.98 86.36 0)
 			(effects
@@
 			)
 		)
-		(property "Footprint" "PCM_marbastlib-mx:SW_MX_HS_CPG151101S11_1u"
+		(property "Footprint" "Macropad:SW_Cherry_MX_PCB_1.00u"
 			(at 73.66 43.18 0)
 			(effects
@@
 			)
 		)
-		(property "Footprint" "PCM_marbastlib-mx:SW_MX_HS_CPG151101S11_1.25u"
+		(property "Footprint" "Macropad:SW_Cherry_MX_PCB_1.25u"
 			(at 114.3 43.18 0)
 			(effects
